Commit message: Made the table bigger to fit all the objects

File: urdf/table.urdf (robot description, URDF)
Before this commit: robot table, 6 links, 5 joints
Links:
- link tabletop: geometry collision box size=2.02 1.02 0.03; visual box size=2.02 1.02 0.03

Commit message: Changed the length of table so that models can fit

File: urdf/table.urdf (robot description, URDF)
Before this commit: robot table, 6 links, 5 joints
Links:
- link tabletop: geometry collision box size=2.02 1.05 0.03; visual box size=2.02 1.05 0.03
